File: estop-driver.sch (KiCad schematic (older format))
At the start: 52 parts, among them J1 Barrel_Jack_Switch, J2 Barrel_Jack_Switch, J3 Conn_01x02, J4 Conn_01x02, J5 Conn_01x02, Q1 BC807, Q2 BC807, Q3 BC817, Q4 BC817, Q5 Q_NMOS_GDS, U1 K7805-2000R3, U2 74HC00, U3 74HC14, U4 74HC02

Commit message: Update KiCad files
Parts:
- removed D1, D18, D19: D, symbol Device:D
- removed D3, D4: LED, LED_SMD:LED_0603_1608Metric_Pad1.05x0.95mm_HandSolder, symbol Device:LED
- removed Q5: Q_NMOS_GDS, symbol Device:Q_NMOS_GDS
- added C1: C, Capacitor_SMD:C_0805_2012Metric_Pad1.15x1.40mm_HandSolder, symbol Device:C
- added D1, D11, D12, D5, D7: LED, LED_SMD:LED_0603_1608Metric_Pad1.05x0.95mm_HandSolder, symbol Device:LED
- added D3, D4: D_Schottky, Diode_SMD:D_SMC, symbol Device:D_Schottky
- added D6: D, Diode_SMD:D_SOD-123, symbol Device:D
- added J1: Conn_01x03, Connector_PinHeader_2.54mm:PinHeader_1x03_P2.54mm_Vertical, symbol Connector_Generic:Conn_01x03
- added Q1, Q6: Q_NMOS_GSD, Package_TO_SOT_SMD:SOT-323_SC-70, symbol Device:Q_NMOS_GSD
- added R22, R25, R4: 2k, Resistor_SMD:R_0603_1608Metric_Pad0.98x0.95mm_HandSolder, symbol Device:R
- added R5: 47, Resistor_SMD:R_0603_1608Metric_Pad0.98x0.95mm_HandSolder, symbol Device:R
- added R6, R7: 10k, Resistor_SMD:R_0603_1608Metric_Pad0.98x0.95mm_HandSolder, symbol Device:R
- added U1: 74HC74, Package_SO:SOIC-14_3.9x8.7mm_P1.27mm, symbol 74xx:74HC74
- added unit 5 of U2
- C5: renamed from C6; footprint (none) -> Capacitor_SMD:C_0805_2012Metric_Pad1.15x1.40mm_HandSolder
- C8: renamed from C7; footprint (none) -> Capacitor_SMD:C_0805_2012Metric_Pad1.15x1.40mm_HandSolder
- C9: renamed from C8; footprint (none) -> Capacitor_SMD:C_0805_2012Metric_Pad1.15x1.40mm_HandSolder
- D2: footprint (none) -> Diode_SMD:D_SOD-123
- D8: renamed from D6; footprint (none) -> Diode_SMD:D_SOD-123
- D9: renamed from D7; footprint (none) -> Diode_SMD:D_SOD-123
- R11: renamed from R7; value R -> 100
- R2: value 10k -> R
- R20: renamed from R16; value R -> 47
- RV1: footprint (none) -> Potentiometer_THT:Potentiometer_Bourns_3296Y_Vertical
- U2: renamed from U3; footprint Package_SO:SO-14_3.9x8.65mm_P1.27mm -> Package_SO:SOIC-14_3.9x8.7mm_P1.27mm
- U3: renamed from U2; footprint Package_SO:SO-14_3.9x8.65mm_P1.27mm -> Package_SO:SOIC-14_3.9x8.7mm_P1.27mm
- U5: renamed from U4; footprint Package_SO:SO-14_3.9x8.65mm_P1.27mm -> Package_SO:SOIC-14_3.9x8.7mm_P1.27mm
- renumbered C1 to C2, C2 to C3, C3 to C4, C4 to C6, C5 to C7, D5 to D10, J1 to J2, J2 to J3, J3 to J4, J4 to J5, J5 to J6, Q1 to Q2, Q2 to Q3, Q3 to Q4, Q4 to Q5, R3 to R10, R8 to R12, R9 to R13, R10 to R14, R11 to R15, R12 to R16, R13 to R17, R14 to R18, R15 to R19, R17 to R21, R18 to R23, R19 to R24, R4 to R3, R5 to R8, R6 to R9, U1 to U4
Connections:
- net GND: now also R1.1, C1.2, J1.3 (Pin_3), Q1.2 (S), Q6.2 (S), R22.1, R25.1, R4.2, R6.1, R7.2; no longer R1.2, R2.2
- net VCC: now also J1.2 (Pin_2), U1.10 (~S), U1.13 (~R), U1.2 (D), U1.4 (~S)
- net estop_od: now also Q1.3 (D), Q6.3 (D)
- net at F1.2: now also D3.1 (K), D4.1 (K); no longer D2.1 (K)
- net control_power_enable: now reaches R23.2, U2.2
- net control_power_enable: now also D11.2 (A)
- net at R20.1, R21.1: now also Q6.1 (G)
- net bat1: now reaches J2.1
- net bat1: now also D2.1 (K), D1.2 (A), D3.2 (A)
- net at D2.2 (A): now also R1.2, D1.1 (K); no longer J3.1
- net thruster_power_enable: now reaches R24.2, U2.6
- net thruster_power_enable: now also D12.2 (A)
- net at R2.1: now also U1.5 (Q)
- net sheet61774296/relay_in renamed sheet6186E17A/relay_2
- net sheet6186E17A/relay_in renamed sheet6186E17A/relay_1
- new net: C1.1, R2.2, U2.11
- new net: U1.1 (~R), U2.10
- new net: J1.1 (Pin_1), U1.12 (D), U1.3 (C)
- new net: Q1.1 (G), R5.1, R7.1
- new net: D7.2 (A), R5.2, U1.9 (Q)
- new net: D7.1 (K), R4.1
- new net: D11.1 (K), R22.2
- new net: D12.1 (K), R25.2
- new net: D5.1 (K), D6.2 (A), R6.2
- new net: U1.11 (C), U1.6 (~Q)
- new net bat2: D4.2 (A), D5.2 (A), D6.1 (K), J3.1
Other:
- moved on the sheet: C2, C3, C4, C5, D10, D8, D9, F1, J2, J3, R10, R3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
