File: kill-switch-reciever.sch (KiCad schematic (older format))
At the start: 8 parts, among them J6 Conn_01x02, Q15 Q_NMOS_GDS, Q16 Q_NMOS_GDS

Commit message: Update KiCad files
Parts:
- removed D14: D_TVS, symbol Device:D_TVS
- removed J6: Conn_01x02, Connector_PinHeader_2.54mm:PinHeader_1x02_P2.54mm_Vertical, symbol Connector_Generic:Conn_01x02
- removed Q15, Q16: Q_NMOS_GDS, symbol Device:Q_NMOS_GDS
- removed R26, R27, R29: 10k, Resistor_SMD:R_0603_1608Metric_Pad0.98x0.95mm_HandSolder, symbol Device:R
- removed R28: 47, Resistor_SMD:R_0603_1608Metric_Pad0.98x0.95mm_HandSolder, symbol Device:R
- added D19, D20, D21, D28, D29: D_TVS, Diode_SMD:D_SMA, symbol Device:D_TVS
- added D22, D23, D24, D30, D31: D, Diode_SMD:D_SOD-123, symbol Device:D
- added D25, D26, D27, D32, D33: LED, LED_SMD:LED_0603_1608Metric_Pad1.05x0.95mm_HandSolder, symbol Device:LED
- added J10, J11, J7, J8, J9: Conn_01x02, Connector_PinHeader_2.54mm:PinHeader_1x02_P2.54mm_Vertical, symbol Connector_Generic:Conn_01x02
- added Q16, Q17, Q18, Q22, Q23, Q24, Q25, Q26, Q29, Q30: Q_NMOS_GSD, Package_TO_SOT_SMD:SOT-323_SC-70, symbol Device:Q_NMOS_GSD
- added Q19, Q20, Q21, Q27, Q28: BC817, Package_TO_SOT_SMD:SOT-23, symbol Transistor_BJT:BC817
- added R32, R34, R36, R50, R52: 1k, Resistor_SMD:R_0603_1608Metric_Pad0.98x0.95mm_HandSolder, symbol Device:R
- added R33, R35, R37, R41, R42, R43, R51, R53, R56, R57: 10k, Resistor_SMD:R_0603_1608Metric_Pad0.98x0.95mm_HandSolder, symbol Device:R
- added R38, R39, R40, R47, R48, R49, R54, R55, R60, R61: 47, Resistor_SMD:R_0603_1608Metric_Pad0.98x0.95mm_HandSolder, symbol Device:R
- added R44, R45, R46, R58, R59: 2k, Resistor_SMD:R_0603_1608Metric_Pad0.98x0.95mm_HandSolder, symbol Device:R
Connections:
- net GND: now also D19.2 (A2), D20.2 (A2), D21.2 (A2), D28.2 (A2), D29.2 (A2), Q16.2 (S), Q17.2 (S), Q18.2 (S), Q22.2 (S), Q23.2 (S), Q24.2 (S), Q25.2 (S), Q26.2 (S), Q29.2 (S), Q30.2 (S), R33.2, R35.2, R37.2, R44.2, R45.2, R46.2, R51.2, R53.2, R58.2, R59.2
- new net: J7.2 (Pin_2), R33.1, R38.2
- new net: D19.1 (A1), Q16.1 (G), R38.1
- new net: D22.1 (K), Q16.3 (D), Q19.1 (B), R41.2
- new net: J7.1 (Pin_1), R32.2
- new net: D22.2 (A), D25.2 (A), Q19.2 (E), R47.2
- new net: Q22.1 (G), R47.1
- new net: D25.1 (K), R44.1
- new net: J8.2 (Pin_2), R35.1, R39.2
- new net: D20.1 (A1), Q17.1 (G), R39.1
- new net: D23.1 (K), Q17.3 (D), Q20.1 (B), R42.2
- new net: J8.1 (Pin_1), R34.2
- new net: D23.2 (A), D26.2 (A), Q20.2 (E), R48.2
- new net: Q23.1 (G), R48.1
- new net: D26.1 (K), R45.1
- new net: J9.2 (Pin_2), R37.1, R40.2
- new net: D21.1 (A1), Q18.1 (G), R40.1
- new net: D24.1 (K), Q18.3 (D), Q21.1 (B), R43.2
- new net: J9.1 (Pin_1), R36.2
- new net: D24.2 (A), D27.2 (A), Q21.2 (E), R49.2
- new net: Q24.1 (G), R49.1
- new net: D27.1 (K), R46.1
- new net: J10.2 (Pin_2), R51.1, R54.2
- new net: D28.1 (A1), Q25.1 (G), R54.1
- new net: D30.1 (K), Q25.3 (D), Q27.1 (B), R56.2
- new net: J10.1 (Pin_1), R50.2
- new net: D30.2 (A), D32.2 (A), Q27.2 (E), R60.2
- new net: Q29.1 (G), R60.1
- new net: D32.1 (K), R58.1
- new net: J11.2 (Pin_2), R53.1, R55.2
- new net: D29.1 (A1), Q26.1 (G), R55.1
- new net: D31.1 (K), Q26.3 (D), Q28.1 (B), R57.2
- new net: J11.1 (Pin_1), R52.2
- new net: D31.2 (A), D33.2 (A), Q28.2 (E), R61.2
- new net: Q30.1 (G), R61.1
- new net: D33.1 (K), R59.1
- new net VCC: Q19.3 (C), Q20.3 (C), Q21.3 (C), Q27.3 (C), Q28.3 (C), R32.1, R34.1, R36.1, R41.1, R42.1, R43.1, R50.1, R52.1, R56.1, R57.1
- new net estop_od_out_1: Q22.3 (D)
- new net estop_od_out_2: Q23.3 (D)
- new net estop_od_out_3: Q24.3 (D)
- new net estop_od_out_4: Q29.3 (D)
- new net estop_od_out_5: Q30.3 (D)
