File: power-relay.sch (KiCad schematic (older format))
At the start: 9 parts, among them K1 G7EB, Q6 BC817, Q7 BC807, Q8 Q_NMOS_GDS

Commit message: Update KiCad files
Parts:
- removed D8: D, symbol Device:D
- removed Q8: Q_NMOS_GDS, symbol Device:Q_NMOS_GDS
- added C11, C12: 100u, Capacitor_SMD:C_Elec_8x5.4, symbol Device:CP
- added D13, D15, D17: D_Schottky, Diode_SMD:D_SMA, symbol Device:D_Schottky
- added D16, D18: D_TVS, Diode_SMD:D_SMA, symbol Device:D_TVS
- added K2, K3: G7EB, MechRelay:G7EB-1A, symbol MechRelay:G7EB
- added Q10, Q13: BC817, Package_TO_SOT_SMD:SOT-23, symbol Transistor_BJT:BC817
- added Q11, Q14: BC807, Package_TO_SOT_SMD:SOT-23, symbol Transistor_BJT:BC807
- added Q12, Q15, Q9: Q_NMOS_GSD, Package_TO_SOT_SMD:SOT-23, symbol Device:Q_NMOS_GSD
- added R28, R30: 47, Resistor_SMD:R_0603_1608Metric_Pad0.98x0.95mm_HandSolder, symbol Device:R
- added R29, R31: 10k, Resistor_SMD:R_0603_1608Metric_Pad0.98x0.95mm_HandSolder, symbol Device:R
- D14: renamed from D9; footprint (none) -> Diode_SMD:D_SMA
- K1: footprint (none) -> MechRelay:G7EB-1A
- R26: renamed from R20; value R -> 47
- R27: renamed from R21; value R -> 10k
- renumbered C9 to C10, Q6 to Q7, Q7 to Q8
Connections:
- net +BATT: now also C11.1, C12.1, D13.1 (K), D15.1 (K), D17.1 (K), K2.2, K3.2
- net GND: now also C11.2, C12.2, D16.2 (A2), D18.2 (A2), Q11.3 (C), Q12.2 (S), Q14.3 (C), Q15.2 (S), Q9.2 (S), R29.2, R31.2
- net VCC: now also Q10.3 (C), Q13.3 (C)
- net at D14.1 (A1), R26.1, R27.1: now also Q9.1 (G)
- net at K1.1: now also D13.2 (A), Q9.3 (D)
- net relay_in renamed relay_1
- new net: Q10.2 (E), Q11.2 (E), R28.2
- new net: D15.2 (A), K2.1, Q12.3 (D)
- new net: D16.1 (A1), Q12.1 (G), R28.1, R29.1
- new net: Q13.2 (E), Q14.2 (E), R30.2
- new net: D17.2 (A), K3.1, Q15.3 (D)
- new net: D18.1 (A1), Q15.1 (G), R30.1, R31.1
- new net relay_2: Q10.1 (B), Q11.1 (B)
- new net relay_3: Q13.1 (B), Q14.1 (B)
Other:
- moved on the sheet: C10, D14, K1, Q7, Q8, R26, R27
